File: manufacturing/MTAP-MIDI-GTCN_V1/MTAP-Embedded.sch (EAGLE design)
At the start: 44 parts, among them IC1 ESP32-WROOM-32UE-N8, IC2 AMS1117-3.3, IC3 PCM1821IRTER, X1 USB4140-GF-0230-C

Commit message: upd analog board
Parts:
- added C16: 10n, rcl_GruS:C-EUC0805
- added C19: 680n, rcl_GruS:C-EUC0805
- added C21: 10n, rcl_GruS:C-EULC0805
- added R12: 6k2, rcl_GruS:R-EU_R0805
- added R13: 2k4, rcl_GruS:R-EUSR0805
- added R14: 240, rcl_GruS:R-EU_R0805
- added R15: 5k1, rcl_GruS:R-EU_R0805
- added R16: 200, rcl_GruS:R-EU_R0805
- added R17: 750, rcl_GruS:R-EU_R0805
- added V4: TLV9354IPWR, opv_GruS:TLV9354IPWR
- added X3: (no value), con-lstb:MA02-1
Connections:
- removed net GPIO17: IC1.IO17
- new net N$10: R14.1, R15.2, V4D.O
- new net N$11: C21.2, R16.2, V4C.P
- new net N$5: R12.1, X3.3
- new net N$6: C16.1, R12.2, V4D.P
- new net N$7: R13.2, R15.1, V4D.N
- new net N$8: C19.1, R14.2, R16.1, R17.1
- net AVDD: now also V4P.VCC
- net FTM0: now also IC1.IO17
- net GND: now also C16.2, C19.2, R13.1, V4C.N, V4P.VSS, X3.2
- net IN1P: now also C21.1, R17.2, V4C.O
Other:
- moved on the sheet: C10, C11, C12, C13, C14, C15, C17, C18, C20, IC3, X2

Commit message: upd pcb
added filter to schematic
Connections:
- net GND: now also V4B.N, V4B.P, V4C.P, V4D.N
- net IN1P: now also V4D.O; no longer V4C.O
- net N$10: now also V4A.O; no longer V4D.O
- net N$11: now also V4D.P; no longer V4C.P
- net N$6: now also V4A.P; no longer V4D.P
- net N$7: now also V4A.N; no longer V4D.N

Commit message: ADC unavailable PCB upd
#3 Issued.
Last Push before replacement.
Parts:
- removed X1: USB4140-GF-0230-C, con_GruS:USB4140-GF-0230-C
- removed X3: (no value), con-lstb:MA02-1
- added J1: 629105150521, Wurth_Connectors_WR-USB:629105150521
Connections:
- removed net IN1M: IC3.IN1M
- net GND: now also IC3.IN1M; no longer X3.2
- net N$5: no longer X3.3
- net PGND: now also J1.GND, J1.SHIELD; no longer X1.GND_1, X1.GND_2, X1.MH1, X1.MH2, X1.MH3, X1.MH4
- net USB_DN: now also J1.D-; no longer X1.CC2
- net USB_DP: now also J1.D+; no longer X1.CC1
- net VBUS: now also J1.VBUS; no longer X1.VBUS_1, X1.VBUS_2

Commit message: New Layout
Parts:
- removed C10, C12: 1u, rcl_GruS:C-EUC0805
- removed C11, C13, C14: 10u, rcl_GruS:C-EUC0805
- removed C15, C17, C18, C20: 100n, rcl_GruS:C-EUC0805
- removed C16: 10n, rcl_GruS:C-EUC0805
- removed C19: 680n, rcl_GruS:C-EUC0805
- removed C21: 10n, rcl_GruS:C-EULC0805
- removed IC3: PCM1821IRTER, adc-dac_GruS:PCM1821IRTER
- removed R12: 6k2, rcl_GruS:R-EU_R0805
- removed R13: 2k4, rcl_GruS:R-EUSR0805
- removed R14: 240, rcl_GruS:R-EU_R0805
- removed R15: 5k1, rcl_GruS:R-EU_R0805
- removed R16: 200, rcl_GruS:R-EU_R0805
- removed R17: 750, rcl_GruS:R-EU_R0805
- removed R3, R4: 0R, rcl_GruS:R-EU_R0805
- removed V4: TLV9354IPWR, opv_GruS:TLV9354IPWR
- removed X2: (no value), con_GruS:JUMPSMD1FACH-1SHORT
- added S3: (no value), switch_GruS:SLIDE_SW
Connections:
- removed net AVDD: C12.1, C18.1, IC3.AVDD, V4P.VCC, X2.2
- removed net IN1P: C21.1, IC3.IN1P, R17.2, V4D.O
- removed net IN2M: IC3.IN2M
- removed net IN2P: IC3.IN2P
- removed net N$10: R14.1, R15.2, V4A.O
- removed net N$11: C21.2, R16.2, V4D.P
- removed net N$13: C11.1, C15.1, IC3.DREG
- removed net N$17: C13.1, C17.1, IC3.AREG
- removed net N$5: R12.1
- removed net N$6: C16.1, R12.2, V4A.P
- removed net N$7: R13.2, R15.1, V4A.N
- removed net N$8: C19.1, R14.2, R16.1, R17.1
- removed net N$9: C10.1, IC3.VREF
- new net RXD1: S3B.S
- new net TXD1: S3A.S
- net +3V3: no longer C14.1, C20.1, IC3.IOVDD, X2.1
- net BCLK: no longer IC3.BCLK
- net FSYNC: no longer IC3.FSYNC
- net FTM0: no longer IC3.FMT0
- net GND: no longer C10.2, C11.2, C12.2, C13.2, C14.2, C15.2, C16.2, C17.2, C18.2, C19.2, C20.2, IC3.IN1M, IC3.VSS_1, IC3.VSS_2, IC3.VSS_3, IC3.VSS_4, IC3.VSS_5, IC3.VSS_6, IC3.VSS_7, IC3.VSS_8, IC3.VSS_9, R13.1, V4B.N, V4B.P, V4C.N, V4C.P, V4D.N, V4P.VSS
- net MD0: no longer IC3.MD0
- net MD1: no longer IC3.MD1
- net MSZ: no longer IC3.MSZ
- net RXD: now also S3A.P; no longer R3.2
- net RXD0: now also S3B.O; no longer R4.1
- net SDATA: no longer IC3.SDOUT
- net TXD: now also S3B.P; no longer R4.2
- net TXD0: now also S3A.O; no longer R3.1
Other:
- note added: "UART Driver 0: Progrqam and Debug UART Driver 1: MIDI Transmission"
